File: channel1.kicad_sch (KiCad schematic)
At the start: 58 parts, among them IC1 TLV73325PDBVT, IC2 TLV73312PDBVT, J2 HDMI-A_Molex_471511001, J3 5051101992, U1 TC358743XBG, U2 TPD8S009DSMR, U3 PCA9517ATP, Y1 Oscillator_27MHz_TXC_7C

Commit message: Switch to micro-HDMI and widely-available parts for JLCPCB
- J2/J4: HDMI-A Molex 471511001 -> micro-HDMI (Type D) Molex 467651001,
  KiCad stock footprint. Symbol renumbered to the Type D pinout.
  D2/D0 fan out on F.Cu; D1/CLK drop to B.Cu via 0.15/0.30 mm vias in
  front of the inner pad row and rejoin the original routing, so the
  ESD-to-TC358743 routing is unchanged. Intra-pair skew re-matched to
  0.000 mm on all 8 pairs. DDC/HPD/CEC/5V re-routed for the new pinout.
- U3/U6: PCA9517ATP (HWSON8) -> PCA9517ADP (MSOP-8, same die), moved
  1.45 mm up into the space freed by the smaller connector.
- Y1/Y2: TXC 7C-27.000MBB-T -> HELE SSI027000E3CH; pads moved to the
  datasheet land (+-1.27 mm, previously +-1.9 mm).
- SP1-4: Wurth 9774060151R -> Sinhoo SMTSO2560CTJ; hole 3.7 -> 4.25 mm.
- IC2/IC4: TLV73312PDBVT -> TLV74312PDBVR (same pinout);
  IC1/IC3: TLV73325PDBVT -> TLV73325PDBVR (reel code).
- 470 pF, 4.7 uF, 2 k, 22 R: MPNs updated to in-stock equivalents.
- Design rules: min via diameter 0.40 -> 0.30 mm,
  min copper-to-edge clearance 0 -> 0.25 mm.

DRC: 0 unconnected, 0 schematic parity issues.

Co-Authored-By: Claude Opus 5.5 <noreply@anthropic.com>
Parts:
- C10, C11, C8, C9: MPN C1608X5R1V475M080AC -> C1608X5R1V475KT000E
- C4, C5, C6, C7: MPN 0402B471K250CT -> CC0402KRX7R9BB471; Manufacturer Walsin -> Yageo
- IC1: value TLV73325PDBVT -> TLV73325PDBVR; symbol antmicroPMICVoltageRegulatorsLinear:TLV73325PDBVT -> antmicroPMICVoltageRegulatorsLinear:TLV73325PDBVR; MPN TLV73325PDBVT -> TLV73325PDBVR
- IC2: value TLV73312PDBVT -> TLV74312PDBVR; symbol antmicroPMICVoltageRegulatorsLinear:TLV73312PDBVT -> antmicroPMICVoltageRegulatorsLinear:TLV74312PDBVR; MPN TLV73312PDBVT -> TLV74312PDBVR
- J2: value HDMI-A_Molex_471511001 -> HDMI-D_Molex_467651001; footprint antmicro-footprints:HDMI-A_Receptacle_Molex_471511001 -> Connector_Video:HDMI_Micro-D_Molex_46765-1xxx; symbol antmicroVideoConnectors:HDMI-A_Molex_471511001 -> antmicroVideoConnectors:HDMI-D_Molex_467651001; MPN 471511001 -> 467651001
- R13: MPN CR0402-FX-22R0GLF -> 0402WGF220JTCE; Manufacturer Bourns -> UNI-ROYAL
- R4: MPN CR0402-FX-2001GLF -> 0402WGF2001TCE; Manufacturer Bourns -> UNI-ROYAL
- U3: value PCA9517ATP -> PCA9517ADP; footprint antmicro-footprints:SOT1069-2 -> Package_SO:MSOP-8_3x3mm_P0.65mm; symbol antmicroLogicTranslatorsLevelShifters:PCA9517ATP -> antmicroLogicTranslatorsLevelShifters:PCA9517ADP; MPN PCA9517ATP -> PCA9517ADP,118
- Y1: value Oscillator_27MHz_TXC_7C -> Oscillator_27MHz_HELE_SSI027000E3CH; symbol antmicroOscillators:Oscillator_27MHz_TXC_7C -> antmicroOscillators:Oscillator_27MHz_HELE_SSI027000E3CH; MPN 7C-27.000MBB-T -> SSI027000E3CH; Manufacturer TXC -> HELE (Harmony Electronics)
Connections:
- net DUMMY1: now also J2.2 (UTILITY/HEAC+); no longer J2.14 (UTILITY/HEAC+)
- net GND: now also J2.10 (D0S), J2.13 (CKS), J2.16 (GND), J2.4 (D2S), J2.7 (D1S); no longer J2.11 (CKS), J2.17 (GND), J2.2 (D2S), J2.5 (D1S), J2.8 (D0S), U3.9 (GND)
- net HDMI1_CEC: now also J2.15 (CEC); no longer J2.13 (CEC)
- net HDMI1_CLK_N: now also J2.14 (CK-); no longer J2.12 (CK-)
- net HDMI1_CLK_P: now also J2.12 (CK+); no longer J2.10 (CK+)
- net HDMI1_D0_N: now also J2.11 (D0-); no longer J2.9 (D0-)
- net HDMI1_D0_P: now also J2.9 (D0+); no longer J2.7 (D0+)
- net HDMI1_D1_N: now also J2.8 (D1-); no longer J2.6 (D1-)
- net HDMI1_D1_P: now also J2.6 (D1+); no longer J2.4 (D1+)
- net HDMI1_D2_N: now also J2.5 (D2-); no longer J2.3 (D2-)
- net HDMI1_D2_P: now also J2.3 (D2+); no longer J2.1 (D2+)
- net HDMI1_DDC_SCL: now also J2.17 (SCL); no longer J2.15 (SCL)
- net HDMI1_DDC_SDA: now also J2.18 (SDA); no longer J2.16 (SDA)
- net HDMI1_HPD: now also J2.1 (HPD/HEAC-); no longer J2.19 (HPD/HEAC-)
- net HDMI1_POWER: now also J2.19 (+5V); no longer J2.18 (+5V)
Changed lines of the file:
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@@
 			)
 		)
-		(property "Description" ""
+		(property "Description" "SMD Multilayer Ceramic Capacitor, 4.7 µF, 35 V, X5R, ±10%, 0603 [1608 Metric]"
 			(at 231.14 228.6 0)
 			(show_name no)
@@
 			)
 		)
-		(property "MPN" "C1608X5R1V475M080AC"
+		(property "MPN" "C1608X5R1V475KT000E"
 			(at 248.92 208.28 0)
 			(hide yes)
@@
 			)
 		)
-		(property "Datasheet" "https://www.passivecomponent.com/wp-content/uploads/datasheet/WTC_MLCC_General_Purpose.pdf"
+		(property "Datasheet" "https://www.yageo.com/upload/media/product/productsearch/datasheet/mlcc/UPY-GPHC_X7R_6.3V-to-50V_18.pdf"
 			(at 204.47 261.62 0)
 			(hide yes)
@@
 			)
 		)
-		(property "Description" ""
+		(property "Description" "SMD Multilayer Ceramic Capacitor, General Purpose, 470 pF, 50 V, X7R, ±10%, 0402 [1005 Metric]"
 			(at 219.71 241.3 0)
 			(show_name no)
@@
 			)
 		)
-		(property "Manufacturer" "Walsin"
+		(property "Manufacturer" "Yageo"
 			(at 199.39 261.62 0)
 			(hide yes)
@@
 			)
 		)
-		(property "MPN" "0402B471K250CT"
+		(property "MPN" "CC0402KRX7R9BB471"
 			(at 201.93 261.62 0)
 			(hide yes)
@@
 			)
 		)
-		(property "Description" ""
+		(property "Description" "SMD Multilayer Ceramic Capacitor, 4.7 µF, 35 V, X5R, ±10%, 0603 [1608 Metric]"
 			(at 231.14 198.12 0)
 			(show_name no)
@@
 			)
 		)
-		(property "MPN" "C1608X5R1V475M080AC"
+		(property "MPN" "C1608X5R1V475KT000E"
 			(at 248.92 177.8 0)
 			(hide yes)
@@
 	)
 	(symbol
-		(lib_id "antmicroPMICVoltageRegulatorsLinear:TLV73312PDBVT")
+		(lib_id "antmicroPMICVoltageRegulatorsLinear:TLV74312PDBVR")
 		(at 331.47 205.74 0)
 		(unit 1)
@@
 			)
 		)
-		(property "Value" "TLV73312PDBVT"
+		(property "Value" "TLV74312PDBVR"
 			(at 334.645 202.565 0)
 			(hide yes)
@@
 			)
 		)
-		(property "Datasheet" "https://www.ti.com/lit/ds/symlink/tlv733p.pdf?HQS=dis-mous-null-mousermode-dsf-pf-null-wwe&ts=1676978230940&ref_url=https%253A%252F%252Fwww.mouser.com%252F"
+		(property "Datasheet" "https://www.ti.com/lit/ds/symlink/tlv743p.pdf"
 			(at 367.03 215.9 0)
 			(hide yes)
@@
 			)
 		)
-		(property "Description" ""
+		(property "Description" "300-mA Low-Dropout Regulator, 1.2 V fixed output, SOT-23-5"
 			(at 331.47 205.74 0)
 			(show_name no)
@@
 			)
 		)
-		(property "MPN" "TLV73312PDBVT"
+		(property "MPN" "TLV74312PDBVR"
 			(at 334.01 202.565 0)
 			(show_name no)
@@
 			)
 		)
-		(property "Datasheet" "https://www.passivecomponent.com/wp-content/uploads/datasheet/WTC_MLCC_General_Purpose.pdf"
+		(property "Datasheet" "https://www.yageo.com/upload/media/product/productsearch/datasheet/mlcc/UPY-GPHC_X7R_6.3V-to-50V_18.pdf"
 			(at 204.47 213.36 0)
 			(hide yes)
@@
 			)
 		)
-		(property "Description" ""
+		(property "Description" "SMD Multilayer Ceramic Capacitor, General Purpose, 470 pF, 50 V, X7R, ±10%, 0402 [1005 Metric]"
 			(at 219.71 193.04 0)
 			(show_name no)
@@
 			)
 		)
-		(property "Manufacturer" "Walsin"
+		(property "Manufacturer" "Yageo"
 			(at 199.39 213.36 0)
 			(hide yes)
@@
 			)
 		)
-		(property "MPN" "0402B471K250CT"
+		(property "MPN" "CC0402KRX7R9BB471"
 			(at 201.93 213.36 0)
 			(hide yes)
@@
 	)
 	(symbol
-		(lib_id "antmicroLogicTranslatorsLevelShifters:PCA9517ATP")
+		(lib_id "antmicroLogicTranslatorsLevelShifters:PCA9517ADP")
 		(at 335.28 97.79 0)
 		(unit 1)
@@
 			)
 		)
-		(property "Value" "PCA9517ATP"
+		(property "Value" "PCA9517ADP"
 			(at 337.82 94.615 0)
 			(hide yes)
@@
 			)
 		)
-		(property "Footprint" "antmicro-footprints:SOT1069-2"
+		(property "Footprint" "Package_SO:MSOP-8_3x3mm_P0.65mm"
 			(at 368.3 105.41 0)
 			(hide yes)
@@
 			)
 		)
-		(property "MPN" "PCA9517ATP"
+		(property "MPN" "PCA9517ADP,118"
 			(at 337.82 94.615 0)
 			(show_name no)
@@
 		(pin "8"
 		)
-		(pin "9"
-		)
 		(instances
 			(project "antmicro-hdmi-mipi-bridge-hw"
@@
 			)
 		)
-		(property "Datasheet" "https://www.passivecomponent.com/wp-content/uploads/datasheet/WTC_MLCC_General_Purpose.pdf"
+		(property "Datasheet" "https://www.yageo.com/upload/media/product/productsearch/datasheet/mlcc/UPY-GPHC_X7R_6.3V-to-50V_18.pdf"
 			(at 204.47 243.84 0)
 			(hide yes)
@@
 			)
 		)
-		(property "Description" ""
+		(property "Description" "SMD Multilayer Ceramic Capacitor, General Purpose, 470 pF, 50 V, X7R, ±10%, 0402 [1005 Metric]"
 			(at 219.71 223.52 0)
 			(show_name no)
@@
 			)
 		)
-		(property "Manufacturer" "Walsin"
+		(property "Manufacturer" "Yageo"
 			(at 199.39 243.84 0)
 			(hide yes)
@@
 			)
 		)
-		(property "MPN" "0402B471K250CT"
+		(property "MPN" "CC0402KRX7R9BB471"
 			(at 201.93 243.84 0)
 			(hide yes)
@@
 	)
 	(symbol
-		(lib_id "antmicroOscillators:Oscillator_27MHz_TXC_7C")
+		(lib_id "antmicroOscillators:Oscillator_27MHz_HELE_SSI027000E3CH")
 		(at 337.82 38.1 0)
 		(unit 1)
@@
 			)
 		)
-		(property "Value" "Oscillator_27MHz_TXC_7C"
+		(property "Value" "Oscillator_27MHz_HELE_SSI027000E3CH"
 			(at 363.22 50.165 0)
 			(hide yes)
@@
 			)
 		)
-		(property "Datasheet" "http://www.txccorp.com/download/products/oscillators/2015TXC_7C_57.pdf"
+		(property "Datasheet" "https://www.lcsc.com/datasheet/lcsc_datasheet_1912111437_HELE-Harmony-Elec-SSI027000E3CH_C254224.pdf"
 			(at 363.22 55.245 0)
 			(hide yes)
@@
 			)
 		)
-		(property "Description" ""
+		(property "Description" "Oscillator, 27 MHz, 25 ppm, SMT, 5mm x 3.2mm, 3.3 V, CMOS"
 			(at 337.82 38.1 0)
 			(show_name no)
@@
 			)
 		)
-		(property "MPN" "7C-27.000MBB-T"
+		(property "MPN" "SSI027000E3CH"
 			(at 338.455 34.925 0)
 			(show_name no)
@@
 			)
 		)
-		(property "Manufacturer" "TXC"
+		(property "Manufacturer" "HELE (Harmony Electronics)"
 			(at 363.22 45.085 0)
 			(hide yes)
@@
 			)
 		)
-		(property "Datasheet" "https://www.bourns.com/docs/product-datasheets/cr.pdf"
+		(property "Datasheet" "https://www.lcsc.com/datasheet/lcsc_datasheet_2206010116_UNI-ROYAL-Uniroyal-Elec-0402WGF220JTCE_C25092.pdf"
 			(at 391.16 55.88 0)
 			(hide yes)
@@
 			)
 		)
-		(property "Manufacturer" "Bourns"
+		(property "Manufacturer" "UNI-ROYAL"
 			(at 391.16 60.96 0)
 			(hide yes)
@@
 			)
 		)
-		(property "MPN" "CR0402-FX-22R0GLF"
+		(property "MPN" "0402WGF220JTCE"
 			(at 391.16 58.42 0)
 			(hide yes)
@@
 			)
 		)
-		(property "Description" ""
+		(property "Description" "SMD Multilayer Ceramic Capacitor, 4.7 µF, 35 V, X5R, ±10%, 0603 [1608 Metric]"
 			(at 231.14 246.38 0)
 			(show_name no)
@@
 			)
 		)
-		(property "MPN" "C1608X5R1V475M080AC"
+		(property "MPN" "C1608X5R1V475KT000E"
 			(at 248.92 226.06 0)
 			(hide yes)
@@
 			)
 		)
-		(property "Datasheet" "https://www.bourns.com/docs/product-datasheets/cr.pdf"
+		(property "Datasheet" "https://www.lcsc.com/datasheet/lcsc_datasheet_2206010130_UNI-ROYAL-Uniroyal-Elec-0402WGF2001TCE_C4109.pdf"
 			(at 134.62 151.13 0)
 			(hide yes)
@@
 			)
 		)
-		(property "Manufacturer" "Bourns"
+		(property "Manufacturer" "UNI-ROYAL"
 			(at 129.54 151.13 0)
 			(hide yes)
@@
 			)
 		)
-		(property "MPN" "CR0402-FX-2001GLF"
+		(property "MPN" "0402WGF2001TCE"
 			(at 132.08 151.13 0)
 			(hide yes)
@@
 			)
 		)
-		(property "Datasheet" "https://www.passivecomponent.com/wp-content/uploads/datasheet/WTC_MLCC_General_Purpose.pdf"
+		(property "Datasheet" "https://www.yageo.com/upload/media/product/productsearch/datasheet/mlcc/UPY-GPHC_X7R_6.3V-to-50V_18.pdf"
 			(at 204.47 228.6 0)
 			(hide yes)
@@
 			)
 		)
-		(property "Description" ""
+		(property "Description" "SMD Multilayer Ceramic Capacitor, General Purpose, 470 pF, 50 V, X7R, ±10%, 0402 [1005 Metric]"
 			(at 219.71 208.28 0)
 			(show_name no)
@@
 			)
 		)
-		(property "Manufacturer" "Walsin"
+		(property "Manufacturer" "Yageo"
 			(at 199.39 228.6 0)
 			(hide yes)
@@
 			)
 		)
-		(property "MPN" "0402B471K250CT"
+		(property "MPN" "CC0402KRX7R9BB471"
 			(at 201.93 228.6 0)
 			(hide yes)
@@
 	)
 	(symbol
-		(lib_id "antmicroPMICVoltageRegulatorsLinear:TLV73325PDBVT")
+		(lib_id "antmicroPMICVoltageRegulatorsLinear:TLV73325PDBVR")
 		(at 331.47 171.45 0)
 		(unit 1)
@@
 			)
 		)
-		(property "Value" "TLV73325PDBVT"
+		(property "Value" "TLV73325PDBVR"
 			(at 334.645 168.275 0)
 			(hide yes)
@@
 			)
 		)
-		(property "MPN" "TLV73325PDBVT"
+		(property "MPN" "TLV73325PDBVR"
 			(at 334.01 168.275 0)
 			(show_name no)
@@
 			)
 		)
-		(property "Description" ""
+		(property "Description" "SMD Multilayer Ceramic Capacitor, 4.7 µF, 35 V, X5R, ±10%, 0603 [1608 Metric]"
 			(at 231.14 213.36 0)
 			(show_name no)
@@
 			)
 		)
-		(property "MPN" "C1608X5R1V475M080AC"
+		(property "MPN" "C1608X5R1V475KT000E"
 			(at 248.92 193.04 0)
 			(hide yes)
@@
 	)
 	(symbol
-		(lib_id "antmicroVideoConnectors:HDMI-A_Molex_471511001")
+		(lib_id "antmicroVideoConnectors:HDMI-D_Molex_467651001")
 		(at 48.26 30.48 0)
 		(unit 1)
@@
 			)
 		)
-		(property "Value" "HDMI-A_Molex_471511001"
+		(property "Value" "HDMI-D_Molex_467651001"
 			(at 93.98 35.56 0)
 			(hide yes)
@@
 			)
 		)
-		(property "Footprint" "antmicro-footprints:HDMI-A_Receptacle_Molex_471511001"
+		(property "Footprint" "Connector_Video:HDMI_Micro-D_Molex_46765-1xxx"
 			(at 93.98 38.1 0)
 			(hide yes)
@@
 			)
 		)
-		(property "Datasheet" "https://tools.molex.com/pdm_docs/sd/471511001_sd.pdf"
+		(property "Datasheet" "https://www.molex.com/pdm_docs/sd/467651001_sd.pdf"
 			(at 93.98 40.64 0)
 			(hide yes)
@@
 			)
 		)
-		(property "Description" ""
+		(property "Description" "Micro HDMI (Type D) Receptacle, 19 Position, Surface Mount, Right Angle; Through Hole shell"
 			(at 48.26 30.48 0)
 			(show_name no)
@@
 			)
 		)
-		(property "MPN" "471511001"
+		(property "MPN" "467651001"
 			(at 55.245 27.305 0)
 			(show_name no)
@@
 			)
 		)
-		(pin "1"
-		)
-		(pin "10"
-		)
-		(pin "11"
+		(pin "3"
 		)
 		(pin "12"
@@
 		(pin "15"
 		)
-		(pin "16"
+		(pin "2"
 		)
 		(pin "17"
@@
 		(pin "18"
 		)
-		(pin "19"
+		(pin "16"
 		)
-		(pin "2"
+		(pin "19"
 		)
-		(pin "3"
+		(pin "1"
 		)
 		(pin "4"
@@
 		(pin "9"
 		)
+		(pin "10"
+		)
+		(pin "11"
+		)
 		(pin "SH"
