File: channel2.kicad_sch (KiCad schematic)
At the start: 58 parts, among them IC3 TLV73325PDBVT, IC4 TLV73312PDBVT, J4 HDMI-A_Molex_471511001, J5 5051101992, U4 TC358743XBG, U5 TPD8S009DSMR, U6 PCA9517ATP, Y2 Oscillator_27MHz_TXC_7C

Commit message: Switch to micro-HDMI and widely-available parts for JLCPCB
- J2/J4: HDMI-A Molex 471511001 -> micro-HDMI (Type D) Molex 467651001,
  KiCad stock footprint. Symbol renumbered to the Type D pinout.
  D2/D0 fan out on F.Cu; D1/CLK drop to B.Cu via 0.15/0.30 mm vias in
  front of the inner pad row and rejoin the original routing, so the
  ESD-to-TC358743 routing is unchanged. Intra-pair skew re-matched to
  0.000 mm on all 8 pairs. DDC/HPD/CEC/5V re-routed for the new pinout.
- U3/U6: PCA9517ATP (HWSON8) -> PCA9517ADP (MSOP-8, same die), moved
  1.45 mm up into the space freed by the smaller connector.
- Y1/Y2: TXC 7C-27.000MBB-T -> HELE SSI027000E3CH; pads moved to the
  datasheet land (+-1.27 mm, previously +-1.9 mm).
- SP1-4: Wurth 9774060151R -> Sinhoo SMTSO2560CTJ; hole 3.7 -> 4.25 mm.
- IC2/IC4: TLV73312PDBVT -> TLV74312PDBVR (same pinout);
  IC1/IC3: TLV73325PDBVT -> TLV73325PDBVR (reel code).
- 470 pF, 4.7 uF, 2 k, 22 R: MPNs updated to in-stock equivalents.
- Design rules: min via diameter 0.40 -> 0.30 mm,
  min copper-to-edge clearance 0 -> 0.25 mm.

DRC: 0 unconnected, 0 schematic parity issues.

Co-Authored-By: Claude Opus 5.5 <noreply@anthropic.com>
Parts:
- C47, C48, C49, C50: MPN 0402B471K250CT -> CC0402KRX7R9BB471; Manufacturer Walsin -> Yageo
- C51, C52, C53, C54: MPN C1608X5R1V475M080AC -> C1608X5R1V475KT000E
- IC3: value TLV73325PDBVT -> TLV73325PDBVR; symbol antmicroPMICVoltageRegulatorsLinear:TLV73325PDBVT -> antmicroPMICVoltageRegulatorsLinear:TLV73325PDBVR; MPN TLV73325PDBVT -> TLV73325PDBVR
- IC4: value TLV73312PDBVT -> TLV74312PDBVR; symbol antmicroPMICVoltageRegulatorsLinear:TLV73312PDBVT -> antmicroPMICVoltageRegulatorsLinear:TLV74312PDBVR; MPN TLV73312PDBVT -> TLV74312PDBVR
- J4: value HDMI-A_Molex_471511001 -> HDMI-D_Molex_467651001; footprint antmicro-footprints:HDMI-A_Receptacle_Molex_471511001 -> Connector_Video:HDMI_Micro-D_Molex_46765-1xxx; symbol antmicroVideoConnectors:HDMI-A_Molex_471511001 -> antmicroVideoConnectors:HDMI-D_Molex_467651001; MPN 471511001 -> 467651001
- R17: MPN CR0402-FX-2001GLF -> 0402WGF2001TCE; Manufacturer Bourns -> UNI-ROYAL
- R26: MPN CR0402-FX-22R0GLF -> 0402WGF220JTCE; Manufacturer Bourns -> UNI-ROYAL
- U6: value PCA9517ATP -> PCA9517ADP; footprint antmicro-footprints:SOT1069-2 -> Package_SO:MSOP-8_3x3mm_P0.65mm; symbol antmicroLogicTranslatorsLevelShifters:PCA9517ATP -> antmicroLogicTranslatorsLevelShifters:PCA9517ADP; MPN PCA9517ATP -> PCA9517ADP,118
- Y2: value Oscillator_27MHz_TXC_7C -> Oscillator_27MHz_HELE_SSI027000E3CH; symbol antmicroOscillators:Oscillator_27MHz_TXC_7C -> antmicroOscillators:Oscillator_27MHz_HELE_SSI027000E3CH; MPN 7C-27.000MBB-T -> SSI027000E3CH; Manufacturer TXC -> HELE (Harmony Electronics)
Connections:
- net DUMMY2: now also J4.2 (UTILITY/HEAC+); no longer J4.14 (UTILITY/HEAC+)
- net GND: now also J4.10 (D0S), J4.13 (CKS), J4.16 (GND), J4.4 (D2S), J4.7 (D1S); no longer J4.11 (CKS), J4.17 (GND), J4.2 (D2S), J4.5 (D1S), J4.8 (D0S), U6.9 (GND)
- net HDMI2_CEC: now also J4.15 (CEC); no longer J4.13 (CEC)
- net HDMI2_CLK_N: now also J4.14 (CK-); no longer J4.12 (CK-)
- net HDMI2_CLK_P: now also J4.12 (CK+); no longer J4.10 (CK+)
- net HDMI2_D0_N: now also J4.11 (D0-); no longer J4.9 (D0-)
- net HDMI2_D0_P: now also J4.9 (D0+); no longer J4.7 (D0+)
- net HDMI2_D1_N: now also J4.8 (D1-); no longer J4.6 (D1-)
- net HDMI2_D1_P: now also J4.6 (D1+); no longer J4.4 (D1+)
- net HDMI2_D2_N: now also J4.5 (D2-); no longer J4.3 (D2-)
- net HDMI2_D2_P: now also J4.3 (D2+); no longer J4.1 (D2+)
- net HDMI2_DDC_SCL: now also J4.17 (SCL); no longer J4.15 (SCL)
- net HDMI2_DDC_SDA: now also J4.18 (SDA); no longer J4.16 (SDA)
- net HDMI2_HPD: now also J4.1 (HPD/HEAC-); no longer J4.19 (HPD/HEAC-)
- net HDMI2_POWER: now also J4.19 (+5V); no longer J4.18 (+5V)
Changed lines of the file:
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@@
 			)
 		)
-		(property "Description" ""
+		(property "Description" "SMD Multilayer Ceramic Capacitor, 4.7 µF, 35 V, X5R, ±10%, 0603 [1608 Metric]"
 			(at 234.95 250.19 0)
 			(show_name no)
@@
 			)
 		)
-		(property "MPN" "C1608X5R1V475M080AC"
+		(property "MPN" "C1608X5R1V475KT000E"
 			(at 252.73 229.87 0)
 			(hide yes)
@@
 			)
 		)
-		(property "Datasheet" "https://www.passivecomponent.com/wp-content/uploads/datasheet/WTC_MLCC_General_Purpose.pdf"
+		(property "Datasheet" "https://www.yageo.com/upload/media/product/productsearch/datasheet/mlcc/UPY-GPHC_X7R_6.3V-to-50V_18.pdf"
 			(at 208.28 283.21 0)
 			(hide yes)
@@
 			)
 		)
-		(property "Description" ""
+		(property "Description" "SMD Multilayer Ceramic Capacitor, General Purpose, 470 pF, 50 V, X7R, ±10%, 0402 [1005 Metric]"
 			(at 223.52 262.89 0)
 			(show_name no)
@@
 			)
 		)
-		(property "Manufacturer" "Walsin"
+		(property "Manufacturer" "Yageo"
 			(at 203.2 283.21 0)
 			(hide yes)
@@
 			)
 		)
-		(property "MPN" "0402B471K250CT"
+		(property "MPN" "CC0402KRX7R9BB471"
 			(at 205.74 283.21 0)
 			(hide yes)
@@
 			)
 		)
-		(property "Description" ""
+		(property "Description" "SMD Multilayer Ceramic Capacitor, 4.7 µF, 35 V, X5R, ±10%, 0603 [1608 Metric]"
 			(at 234.95 219.71 0)
 			(show_name no)
@@
 			)
 		)
-		(property "MPN" "C1608X5R1V475M080AC"
+		(property "MPN" "C1608X5R1V475KT000E"
 			(at 252.73 199.39 0)
 			(hide yes)
@@
 			)
 		)
-		(property "Datasheet" "https://www.bourns.com/docs/product-datasheets/cr.pdf"
+		(property "Datasheet" "https://www.lcsc.com/datasheet/lcsc_datasheet_2206010116_UNI-ROYAL-Uniroyal-Elec-0402WGF220JTCE_C25092.pdf"
 			(at 393.7 57.15 0)
 			(hide yes)
@@
 			)
 		)
-		(property "Manufacturer" "Bourns"
+		(property "Manufacturer" "UNI-ROYAL"
 			(at 393.7 62.23 0)
 			(hide yes)
@@
 			)
 		)
-		(property "MPN" "CR0402-FX-22R0GLF"
+		(property "MPN" "0402WGF220JTCE"
 			(at 393.7 59.69 0)
 			(hide yes)
@@
 			)
 		)
-		(property "Datasheet" "https://www.passivecomponent.com/wp-content/uploads/datasheet/WTC_MLCC_General_Purpose.pdf"
+		(property "Datasheet" "https://www.yageo.com/upload/media/product/productsearch/datasheet/mlcc/UPY-GPHC_X7R_6.3V-to-50V_18.pdf"
 			(at 208.28 265.43 0)
 			(hide yes)
@@
 			)
 		)
-		(property "Description" ""
+		(property "Description" "SMD Multilayer Ceramic Capacitor, General Purpose, 470 pF, 50 V, X7R, ±10%, 0402 [1005 Metric]"
 			(at 223.52 245.11 0)
 			(show_name no)
@@
 			)
 		)
-		(property "Manufacturer" "Walsin"
+		(property "Manufacturer" "Yageo"
 			(at 203.2 265.43 0)
 			(hide yes)
@@
 			)
 		)
-		(property "MPN" "0402B471K250CT"
+		(property "MPN" "CC0402KRX7R9BB471"
 			(at 205.74 265.43 0)
 			(hide yes)
@@
 	)
 	(symbol
-		(lib_id "antmicroPMICVoltageRegulatorsLinear:TLV73312PDBVT")
+		(lib_id "antmicroPMICVoltageRegulatorsLinear:TLV74312PDBVR")
 		(at 334.01 207.01 0)
 		(unit 1)
@@
 			)
 		)
-		(property "Value" "TLV73312PDBVT"
+		(property "Value" "TLV74312PDBVR"
 			(at 336.55 203.835 0)
 			(hide yes)
@@
 			)
 		)
-		(property "Datasheet" "https://www.ti.com/lit/ds/symlink/tlv733p.pdf?HQS=dis-mous-null-mousermode-dsf-pf-null-wwe&ts=1676978230940&ref_url=https%253A%252F%252Fwww.mouser.com%252F"
+		(property "Datasheet" "https://www.ti.com/lit/ds/symlink/tlv743p.pdf"
 			(at 369.57 217.17 0)
 			(hide yes)
@@
 			)
 		)
-		(property "Description" ""
+		(property "Description" "300-mA Low-Dropout Regulator, 1.2 V fixed output, SOT-23-5"
 			(at 334.01 207.01 0)
 			(show_name no)
@@
 			)
 		)
-		(property "MPN" "TLV73312PDBVT"
+		(property "MPN" "TLV74312PDBVR"
 			(at 336.55 203.835 0)
 			(show_name no)
@@
 	)
 	(symbol
-		(lib_id "antmicroLogicTranslatorsLevelShifters:PCA9517ATP")
+		(lib_id "antmicroLogicTranslatorsLevelShifters:PCA9517ADP")
 		(at 337.82 99.06 0)
 		(unit 1)
@@
 			)
 		)
-		(property "Value" "PCA9517ATP"
+		(property "Value" "PCA9517ADP"
 			(at 340.995 95.885 0)
 			(show_name no)
@@
 			)
 		)
-		(property "Footprint" "antmicro-footprints:SOT1069-2"
+		(property "Footprint" "Package_SO:MSOP-8_3x3mm_P0.65mm"
 			(at 370.84 106.68 0)
 			(hide yes)
@@
 			)
 		)
-		(property "MPN" "PCA9517ATP"
+		(property "MPN" "PCA9517ADP,118"
 			(at 370.84 111.76 0)
 			(hide yes)
@@
 		(pin "8"
 		)
-		(pin "9"
-		)
 		(instances
 			(project "antmicro-hdmi-mipi-bridge-hw"
@@
 			)
 		)
-		(property "Description" ""
+		(property "Description" "SMD Multilayer Ceramic Capacitor, 4.7 µF, 35 V, X5R, ±10%, 0603 [1608 Metric]"
 			(at 234.95 234.95 0)
 			(show_name no)
@@
 			)
 		)
-		(property "MPN" "C1608X5R1V475M080AC"
+		(property "MPN" "C1608X5R1V475KT000E"
 			(at 252.73 214.63 0)
 			(hide yes)
@@
 			)
 		)
-		(property "Datasheet" "https://www.passivecomponent.com/wp-content/uploads/datasheet/WTC_MLCC_General_Purpose.pdf"
+		(property "Datasheet" "https://www.yageo.com/upload/media/product/productsearch/datasheet/mlcc/UPY-GPHC_X7R_6.3V-to-50V_18.pdf"
 			(at 208.28 234.95 0)
 			(hide yes)
@@
 			)
 		)
-		(property "Description" ""
+		(property "Description" "SMD Multilayer Ceramic Capacitor, General Purpose, 470 pF, 50 V, X7R, ±10%, 0402 [1005 Metric]"
 			(at 223.52 214.63 0)
 			(show_name no)
@@
 			)
 		)
-		(property "Manufacturer" "Walsin"
+		(property "Manufacturer" "Yageo"
 			(at 203.2 234.95 0)
 			(hide yes)
@@
 			)
 		)
-		(property "MPN" "0402B471K250CT"
+		(property "MPN" "CC0402KRX7R9BB471"
 			(at 205.74 234.95 0)
 			(hide yes)
@@
 	)
 	(symbol
-		(lib_id "antmicroPMICVoltageRegulatorsLinear:TLV73325PDBVT")
+		(lib_id "antmicroPMICVoltageRegulatorsLinear:TLV73325PDBVR")
 		(at 334.01 173.99 0)
 		(unit 1)
@@
 			)
 		)
-		(property "Value" "TLV73325PDBVT"
+		(property "Value" "TLV73325PDBVR"
 			(at 336.55 170.815 0)
 			(hide yes)
@@
 			)
 		)
-		(property "MPN" "TLV73325PDBVT"
+		(property "MPN" "TLV73325PDBVR"
 			(at 336.55 170.815 0)
 			(show_name no)
@@
 	)
 	(symbol
-		(lib_id "antmicroOscillators:Oscillator_27MHz_TXC_7C")
+		(lib_id "antmicroOscillators:Oscillator_27MHz_HELE_SSI027000E3CH")
 		(at 340.36 39.37 0)
 		(unit 1)
@@
 			)
 		)
-		(property "Value" "Oscillator_27MHz_TXC_7C"
+		(property "Value" "Oscillator_27MHz_HELE_SSI027000E3CH"
 			(at 365.76 51.435 0)
 			(hide yes)
@@
 			)
 		)
-		(property "Datasheet" "http://www.txccorp.com/download/products/oscillators/2015TXC_7C_57.pdf"
+		(property "Datasheet" "https://www.lcsc.com/datasheet/lcsc_datasheet_1912111437_HELE-Harmony-Elec-SSI027000E3CH_C254224.pdf"
 			(at 365.76 56.515 0)
 			(hide yes)
@@
 			)
 		)
-		(property "Description" ""
+		(property "Description" "Oscillator, 27 MHz, 25 ppm, SMT, 5mm x 3.2mm, 3.3 V, CMOS"
 			(at 340.36 39.37 0)
 			(show_name no)
@@
 			)
 		)
-		(property "MPN" "7C-27.000MBB-T"
+		(property "MPN" "SSI027000E3CH"
 			(at 340.995 36.195 0)
 			(show_name no)
@@
 			)
 		)
-		(property "Manufacturer" "TXC"
+		(property "Manufacturer" "HELE (Harmony Electronics)"
 			(at 365.76 46.355 0)
 			(hide yes)
@@
 			)
 		)
-		(property "Datasheet" "https://www.passivecomponent.com/wp-content/uploads/datasheet/WTC_MLCC_General_Purpose.pdf"
+		(property "Datasheet" "https://www.yageo.com/upload/media/product/productsearch/datasheet/mlcc/UPY-GPHC_X7R_6.3V-to-50V_18.pdf"
 			(at 208.28 250.19 0)
 			(hide yes)
@@
 			)
 		)
-		(property "Description" ""
+		(property "Description" "SMD Multilayer Ceramic Capacitor, General Purpose, 470 pF, 50 V, X7R, ±10%, 0402 [1005 Metric]"
 			(at 223.52 229.87 0)
 			(show_name no)
@@
 			)
 		)
-		(property "Manufacturer" "Walsin"
+		(property "Manufacturer" "Yageo"
 			(at 203.2 250.19 0)
 			(hide yes)
@@
 			)
 		)
-		(property "MPN" "0402B471K250CT"
+		(property "MPN" "CC0402KRX7R9BB471"
 			(at 205.74 250.19 0)
 			(hide yes)
@@
 			)
 		)
-		(property "Description" ""
+		(property "Description" "SMD Multilayer Ceramic Capacitor, 4.7 µF, 35 V, X5R, ±10%, 0603 [1608 Metric]"
 			(at 234.95 267.97 0)
 			(show_name no)
@@
 			)
 		)
-		(property "MPN" "C1608X5R1V475M080AC"
+		(property "MPN" "C1608X5R1V475KT000E"
 			(at 252.73 247.65 0)
 			(hide yes)
@@
 	)
 	(symbol
-		(lib_id "antmicroVideoConnectors:HDMI-A_Molex_471511001")
+		(lib_id "antmicroVideoConnectors:HDMI-D_Molex_467651001")
 		(at 50.8 31.75 0)
 		(unit 1)
@@
 			)
 		)
-		(property "Value" "HDMI-A_Molex_471511001"
+		(property "Value" "HDMI-D_Molex_467651001"
 			(at 96.52 36.83 0)
 			(hide yes)
@@
 			)
 		)
-		(property "Footprint" "antmicro-footprints:HDMI-A_Receptacle_Molex_471511001"
+		(property "Footprint" "Connector_Video:HDMI_Micro-D_Molex_46765-1xxx"
 			(at 96.52 39.37 0)
 			(hide yes)
@@
 			)
 		)
-		(property "Datasheet" "https://tools.molex.com/pdm_docs/sd/471511001_sd.pdf"
+		(property "Datasheet" "https://www.molex.com/pdm_docs/sd/467651001_sd.pdf"
 			(at 96.52 41.91 0)
 			(hide yes)
@@
 			)
 		)
-		(property "Description" ""
+		(property "Description" "Micro HDMI (Type D) Receptacle, 19 Position, Surface Mount, Right Angle; Through Hole shell"
 			(at 50.8 31.75 0)
 			(show_name no)
@@
 			)
 		)
-		(property "MPN" "471511001"
+		(property "MPN" "467651001"
 			(at 58.42 27.94 0)
 			(show_name no)
@@
 			)
 		)
-		(pin "1"
-		)
-		(pin "10"
-		)
-		(pin "11"
+		(pin "3"
 		)
 		(pin "12"
@@
 		(pin "15"
 		)
-		(pin "16"
+		(pin "2"
 		)
 		(pin "17"
@@
 		(pin "18"
 		)
-		(pin "19"
+		(pin "16"
 		)
-		(pin "2"
+		(pin "19"
 		)
-		(pin "3"
+		(pin "1"
 		)
 		(pin "4"
@@
 		(pin "9"
 		)
+		(pin "10"
+		)
+		(pin "11"
+		)
 		(pin "SH"
 		)
@@
 			)
 		)
-		(property "Datasheet" "https://www.bourns.com/docs/product-datasheets/cr.pdf"
+		(property "Datasheet" "https://www.lcsc.com/datasheet/lcsc_datasheet_2206010130_UNI-ROYAL-Uniroyal-Elec-0402WGF2001TCE_C4109.pdf"
 			(at 173.99 172.72 0)
 			(hide yes)
@@
 			)
 		)
-		(property "Manufacturer" "Bourns"
+		(property "Manufacturer" "UNI-ROYAL"
 			(at 179.07 172.72 0)
 			(hide yes)
@@
 			)
 		)
-		(property "MPN" "CR0402-FX-2001GLF"
+		(property "MPN" "0402WGF2001TCE"
 			(at 176.53 172.72 0)
 			(hide yes)
